Commit message: add caster wheels with motion

File: catkin_ws/src/urdf_testing/urdf/test_robot.urdf (robot description, URDF)
Before this commit: robot myfirst, 1 links, 0 joints
Links:
- added link c_back; collision sphere radius=0.127; visual sphere radius=0.127
- added link c_front; collision sphere radius=0.127; visual sphere radius=0.127
- added link link_rotate1; collision box size=0.4878 0.8382 0.0381; visual box size=0.4878 0.8382 0.0381
- added link link_rotate2; collision box size=0.4878 0.8382 0.0381; visual box size=0.4878 0.8382 0.0381
- added link wheel_left; collision cylinder length=0.0889 radius=0.127; visual cylinder length=0.0889 radius=0.127
- added link wheel_right; collision cylinder length=0.0889 radius=0.127; visual cylinder length=0.0889 radius=0.127
- link base_link: geometry collision box size=0.4878 0.8382 0.0381; visual box size=0.4878 0.8382 0.0381
Joints:
- added joint base_to_rotate_1: type fixed, parent base_link, child link_rotate1, origin xyz=0 0 0
- added joint base_to_rotate_2: type fixed, parent base_link, child link_rotate2, origin xyz=0 0 0
- added joint joint_c_back: type fixed, parent base_link, child c_back, origin xyz=0 0 0
- added joint joint_c_front: type fixed, parent base_link, child c_front, origin xyz=0 0 0
- added joint w_left: type continuous, parent base_link, child wheel_left, origin xyz=0 0 -0.0254, axis 0 1 0
- added joint w_right: type continuous, parent base_link, child wheel_right, origin xyz=0 0 -0.0254, axis 0 1 0

Commit message: stuff

File: catkin_ws/src/urdf_testing/urdf/test_robot.urdf (robot description, URDF)
Before this commit: robot myfirst, 7 links, 6 joints
Links:
- added link camera_link, mass 1e-5; collision box size=0.05 0.05 0.05; visual box size=0.05 0.05 0.05
- link c_back: geometry collision sphere length=0.0889 radius=0.127; visual sphere length=0.0889 radius=0.127
- link c_front: geometry collision sphere length=0.0889 radius=0.127; visual sphere length=0.0889 radius=0.127
Joints:
- added joint camera_joint: type fixed, parent base_link, child camera_link, origin xyz=0 0 1.5 rpy=0 0 0, axis 0 1 0
- joint joint_c_back: axis (none) -> 0 1 0; origin xyz=0 0 0 -> xyz=-0.3175 0 0 rpy=1.5708 0 0
- joint joint_c_front: axis (none) -> 0 1 0; origin xyz=0 0 0 -> xyz=0.3175 0 0 rpy=1.5708 0 0
- joint w_left: origin xyz=0 0 -0.0254 -> xyz=0 -0.3175 0 rpy=1.5708 0 0; type continuous -> fixed
- joint w_right: origin xyz=0 0 -0.0254 -> xyz=0 0.3175 0 rpy=1.5708 0 0; type continuous -> fixed

Commit message: made it work

File: catkin_ws/src/urdf_testing/urdf/test_robot.urdf (robot description, URDF)
Before this commit: robot myfirst, 8 links, 7 joints
Links:
- link c_back: mass None -> 1
- link c_front: mass None -> 1
- link camera_link: mass 1e-5 -> .1
- link wheel_left: mass None -> 1
- link wheel_right: mass None -> 1
Joints:
- joint camera_joint: origin xyz=0 0 1.5 rpy=0 0 0 -> xyz=0 0 .1 rpy=0 0 0
- joint joint_c_back: type fixed -> continuous
- joint joint_c_front: type fixed -> continuous
- joint w_left: axis 0 1 0 -> 0 0 1; type fixed -> continuous
- joint w_right: axis 0 1 0 -> 0 0 1; type fixed -> continuous

Commit message: getting planning started

File: catkin_ws/src/urdf_testing/urdf/test_robot.urdf (robot description, URDF)
Before this commit: robot myfirst, 8 links, 7 joints
Links:
- removed link camera_link
- removed link wheel_left
- removed link wheel_right
- added link laser_object, mass 0.2; collision cylinder length=0.07 radius=0.06; visual cylinder length=0.07 radius=0.06
- added link link_left_wheel, mass 0.2; collision cylinder length=0.0889 radius=0.127; visual cylinder length=0.0889 radius=0.127
- added link link_right_wheel, mass 0.2; collision cylinder length=0.0889 radius=0.127; visual cylinder length=0.0889 radius=0.127
- link base_link: mass None -> 5
- link c_back: geometry collision sphere length=0.0889 radius=0.1263; visual sphere length=0.0889 radius=0.1263
- link c_front: geometry collision sphere length=0.0889 radius=0.1263; visual sphere length=0.0889 radius=0.1263
Joints:
- removed joint camera_joint
- removed joint w_left
- removed joint w_right
- added joint joint_left_wheel: type continuous, parent base_link, child link_right_wheel, origin xyz=0 -0.3175 0 rpy=0 0 0, axis 0 1 0, limit effort=10000 velocity=1000
- added joint joint_right_wheel: type continuous, parent base_link, child link_left_wheel, origin xyz=0 0.3175 0 rpy=0 0 0, axis 0 1 0, limit effort=10000 velocity=1000
- added joint laser_joint: type fixed, parent base_link, child laser_object, origin xyz=0 0 0.5 rpy=0 0 0
- joint joint_c_back: type continuous -> fixed
- joint joint_c_front: type continuous -> fixed
